Commit message: first prototype of doing callibration and tracking using the three cameras.

File: python/mim_robots/robots/kuka/urdf/iiwa_pusher.urdf (robot description, URDF)
Before this commit: robot KUKAiiwa14, 14 links, 13 joints
Links:
- added link pusher; collision cylinder length=.1 radius=0.02; visual cylinder length=0.1 radius=0.02
- link contact: geometry collision sphere radius=0.00873; visual sphere radius=0.00873
- link kuka_to_sensor_mount: geometry collision mesh filename=package://meshes/kuka/kuka_to_sensor_mount.stl scale=0.001 0.001 0.001; visual mesh filename=package://meshes/kuka/kuka_to_sensor_mount.stl scale=0.001 0.001 0.001
Joints:
- added joint kuka_to_pusher: type fixed, parent L7, child pusher, origin xyz=0 0 0.045 rpy=0 0 0, limit lower=-10 upper=10 effort=1000 velocity=1000
