Commit message: add all files for demo for alex

File: python/mim_robots/robots/kuka/urdf/iiwa_ft_sensor_ball.urdf (robot description, URDF)
Before this commit: robot KUKAiiwa14, 14 links, 13 joints
Links:
- link contact: geometry collision sphere radius=0.00873; visual sphere radius=0.00873
- link kuka_to_sensor_mount: geometry collision mesh filename=package://meshes/kuka/kuka_to_sensor_mount.stl scale=0.001 0.001 0.001; visual mesh filename=package://meshes/kuka/kuka_to_sensor_mount.stl scale=0.001 0.001 0.001
